File: hw/Kicad/supply_and_charger.sch (KiCad schematic (older format))
At the start: 51 parts, among them J201 USB_B_Micro, J202 LIPO 1S, SW1 SW_SPDT, U201 LMR62421XMF, U202 TPS63001, U203 MCP73871-2CC

Commit message: V1.1 version. UART fixed and some signals renamed
Connections:
- net PW_STATE3 is gone; now on net PW_STATE2: R211.2, U203.7 (STAT2)
- net PW_STATE2: no longer R212.2, U203.8 (STAT1/~LBO~)
- net SLEEP renamed SLEEP_12V
- new net PW_STATE1: R212.2, U203.8 (STAT1/~LBO~)
Changed lines of the file:
@@
 Sheet 2 3
 Title "time2time project"
-Date "2019-09-09"
-Rev "V1.0"
+Date "2019-10-29"
+Rev "V1.1"
 Comp "Puma Pride Robotics Team"
 Comment1 "Designed by Rubén Espino San José"
@@
 Text Label 4050 3400 0    50   ~ 0
 USB4
+Text Label 10200 2700 2    50   ~ 0
+PW_STATE1
+Text Label 10200 2800 2    50   ~ 0
+PW_STATE2
 Text Label 10200 2500 2    50   ~ 0
-PW_STATE1
-Text Label 10200 2700 2    50   ~ 0
-PW_STATE2
-Text Label 10200 2800 2    50   ~ 0
 PW_STATE3
 Connection ~ 3300 1750
@@
 Connection ~ 2400 6550
 Text HLabel 1550 6550 0    50   Input ~ 0
-SLEEP
+SLEEP_12V
 NoConn ~ 3000 4050
 $Comp
